File: gaspmask.sch (EAGLE design)
At the start: 9 parts, among them IC1 PIC12F629P, U1 BMP180

Commit message: Revised to take cheap chinese daughter board.
Parts:
- added JP4: (no value), SparkFun-Connectors:M04LOCK_LONGPADS
Connections:
- removed net N$4: IC1.GP2, U1.SCL
- removed net N$5: IC1.GP1, U1.SDA
- new net SCL: IC1.GP2, JP4.3, U1.SCL
- new net SDA: IC1.GP1, JP4.4, U1.SDA
- net +5V: now also JP4.1
- net GND: now also JP4.2
Changed lines of the file:
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@@
 <part name="P+5" library="supply1" deviceset="+5V" device=""/>
 <part name="JP3" library="SparkFun-Connectors" deviceset="M02" device="-JST-2-PTH-NO_SILK"/>
+<part name="JP4" library="SparkFun-Connectors" deviceset="M04" device="LOCK_LONGPADS"/>
 </parts>
 <sheets>
@@
 <instance part="P+5" gate="1" x="152.4" y="58.42"/>
 <instance part="JP3" gate="G$1" x="-10.16" y="81.28"/>
+<instance part="JP4" gate="G$1" x="109.22" y="17.78"/>
 </instances>
 <busses>
@@
 <pinref part="JP3" gate="G$1" pin="1"/>
 <wire x1="0" y1="81.28" x2="-2.54" y2="81.28" width="0.1524" layer="91"/>
+</segment>
+<segment>
+<pinref part="JP4" gate="G$1" pin="2"/>
+<wire x1="114.3" y1="17.78" x2="129.54" y2="17.78" width="0.1524" layer="91"/>
+<label x="119.38" y="17.78" size="1.778" layer="95"/>
 </segment>
 </net>
@@
 <wire x1="0" y1="83.82" x2="0" y2="86.36" width="0.1524" layer="91"/>
 </segment>
+<segment>
+<pinref part="JP4" gate="G$1" pin="1"/>
+<wire x1="129.54" y1="15.24" x2="114.3" y2="15.24" width="0.1524" layer="91"/>
+<label x="119.38" y="15.24" size="1.778" layer="95"/>
+</segment>
 </net>
 <net name="N$2" class="0">
@@
 <pinref part="JP1" gate="G$1" pin="2"/>
 <wire x1="55.88" y1="48.26" x2="25.4" y2="48.26" width="0.1524" layer="91"/>
-</segment>
-</net>
-<net name="N$4" class="0">
-<segment>
-<pinref part="IC1" gate="G$1" pin="GP2"/>
-<pinref part="U1" gate="G$1" pin="SCL"/>
-<wire x1="99.06" y1="45.72" x2="119.38" y2="45.72" width="0.1524" layer="91"/>
-</segment>
-</net>
-<net name="N$5" class="0">
-<segment>
-<pinref part="U1" gate="G$1" pin="SDA"/>
-<pinref part="IC1" gate="G$1" pin="GP1"/>
-<wire x1="119.38" y1="50.8" x2="99.06" y2="50.8" width="0.1524" layer="91"/>
 </segment>
 </net>
@@
 </segment>
 </net>
+<net name="SDA" class="0">
+<segment>
+<pinref part="JP4" gate="G$1" pin="4"/>
+<wire x1="114.3" y1="22.86" x2="129.54" y2="22.86" width="0.1524" layer="91"/>
+<label x="119.38" y="22.86" size="1.778" layer="95"/>
+</segment>
+<segment>
+<pinref part="U1" gate="G$1" pin="SDA"/>
+<pinref part="IC1" gate="G$1" pin="GP1"/>
+<wire x1="119.38" y1="50.8" x2="99.06" y2="50.8" width="0.1524" layer="91"/>
+<label x="104.14" y="50.8" size="1.778" layer="95"/>
+</segment>
+</net>
+<net name="SCL" class="0">
+<segment>
+<pinref part="JP4" gate="G$1" pin="3"/>
+<wire x1="129.54" y1="20.32" x2="114.3" y2="20.32" width="0.1524" layer="91"/>
+<label x="119.38" y="20.32" size="1.778" layer="95"/>
+</segment>
+<segment>
+<pinref part="IC1" gate="G$1" pin="GP2"/>
+<pinref part="U1" gate="G$1" pin="SCL"/>
+<wire x1="99.06" y1="45.72" x2="119.38" y2="45.72" width="0.1524" layer="91"/>
+<label x="104.14" y="45.72" size="1.778" layer="95"/>
+</segment>
+</net>
